File: ch32m030/ch32m030.kicad_pcb (KiCad board)
At the start: 4 copper layers, 65.5 x 100.3 mm, 139 parts, among them J1 TBL002A-350-10GY-2GY, J2 Connector, USB-TYPE-C-16P, J3 691256610006, J4 SM06B-SRSS-TBLFSN, P1 2204061-2 Edge Connector, Q1 BSC019N06NSATMA1, Q2 BSC019N06NSATMA1, Q3 BSC019N06NSATMA1, Q4 BSC019N06NSATMA1, Q5 BSC019N06NSATMA1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

Commit message: v1
Parts:
- removed FB1: ~, PCM_JLCPCB:FB_0603
- moved R20 13.0 mm to (165.6, 121.0)
- moved R8 11.2 mm to (165.0, 93.2)
Connections:
- C12 pad 2: GNDPWR -> GND
- C13 pad 2: GNDPWR -> GND
- C18 pad 2: GNDPWR -> GND
- C19 pad 2: GNDPWR -> GND
- C24 pad 2: GNDPWR -> GND
- C25 pad 2: GNDPWR -> GND
- C6 pad 2: GNDPWR -> GND
- C7 pad 2: GNDPWR -> GND
- J2 pad A12B1: GNDPWR -> GND
- J2 pad B12A1: GNDPWR -> GND
- J2 pad S1: GNDPWR -> GND
- J3 pad 6: GNDPWR -> GND
- J3 pad A6: GNDPWR -> GND
- P1 pad 39: GNDPWR -> GND
- P1 pad 40: GNDPWR -> GND
- R19 pad 2: GNDPWR -> GND
- R20 pad 2: GNDPWR -> GND
- R57 pad 2: GNDPWR -> GND
- R59 pad 2: GNDPWR -> GND
- R7 pad 2: GNDPWR -> GND
- R8 pad 2: GNDPWR -> GND
Routing:
- net GNDPWR: track 56.0 -> 0.00 mm, vias 97 -> 0
- net GND: vias 66 -> 158
- net +24V: vias 52 -> 51
- added copper zone on In2.Cu, net GND
- removed copper zone on B.Cu, net GNDPWR
- removed copper zone on F.Cu, net GNDPWR
- removed copper zone on In1.Cu, net GNDPWR
- removed copper zone on In2.Cu, net GNDPWR

Commit message: update board
Parts:
- C28, C29, C30, C31, R29, R30, R31, R32, R33, R34, R35, R36, R37, R38, R39, R40: moved to B.Cu
- moved R37 44.1 mm to (114.0, 121.4), turned to 0 degrees
- moved R40 44.0 mm to (113.8, 86.8), turned to 180 degrees
- moved R39 44.0 mm to (113.8, 101.2), turned to 0 degrees
- moved R36 42.9 mm to (114.0, 120.0), turned to 0 degrees
- moved R33 42.8 mm to (113.8, 88.2), turned to 180 degrees
- moved R34 42.5 mm to (113.8, 99.8), turned to 0 degrees
- moved R38 41.9 mm to (113.2, 107.2), turned to 180 degrees
- moved R32 41.7 mm to (114.0, 118.6), turned to 180 degrees
- moved R29 41.7 mm to (113.8, 89.6), turned to 0 degrees
- moved R30 41.0 mm to (113.8, 98.4), turned to 180 degrees
- moved C31 40.6 mm to (114.0, 117.2), turned to 180 degrees
- moved C28 40.5 mm to (113.8, 91.0), turned to 0 degrees
- moved R35 40.4 mm to (113.2, 108.6), turned to 180 degrees
- moved C29 39.6 mm to (113.8, 97.0), turned to 180 degrees
- moved R31 38.9 mm to (113.2, 110.0), turned to 0 degrees
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Routing:
- net /LIM_H: track 114.6 -> 0.00 mm, vias 4 -> 0
- net /LIM_L: track 110.4 -> 0.00 mm, vias 4 -> 0
- net /SW3: track 96.7 -> 0.00 mm, vias 37 -> 0
- net /BRAKE: track 92.4 -> 0.00 mm, vias 3 -> 0
- net +24V: track 85.5 -> 0.00 mm, vias 51 -> 0
- net GND: track 85.0 -> 0.00 mm, vias 158 -> 0
- net /RST: track 79.7 -> 0.00 mm, vias 3 -> 0
- net /SW2: track 79.1 -> 0.00 mm, vias 37 -> 0
- net /BEMF_X: track 78.8 -> 0.00 mm, vias 5 -> 0
- net /fets/VGH3: track 77.0 -> 0.00 mm, vias 2 -> 0
- net /BEMF_C: track 73.7 -> 0.00 mm, vias 5 -> 0
- net /BEMF_W: track 73.6 -> 0.00 mm, vias 5 -> 0
- net /IS_2_P: track 72.4 -> 0.00 mm, vias 3 -> 0
- net /SPI_MISO: track 70.4 -> 0.00 mm, vias 4 -> 0
- net /fets/VGL3: track 70.0 -> 0.00 mm, vias 2 -> 0
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