File: ch32m030/ch32m030.kicad_sch (KiCad schematic)
At the start: 50 parts, among them J1 TBL002A-350-10GY-2GY, J3 691256610006, J4 SM06B-SRSS-TBLFSN, P1 2204061-2 Edge Connector, U1 CH32M030C8U3, U2 HT7533, X1 X50328MSB2GI

Commit message: v1
Parts:
- removed FB1: ~, PCM_JLCPCB:FB_0603, symbol PCM_JLCPCB-Inductors:Ferrite,0603
Connections:
- net GNDPWR is gone; now on net GND: J3.6, J3.A6, P1.39 (P3), P1.40 (P4)

Commit message: update board
Connections:
- net SYNC: no longer D6.3 (I/O)
Changed lines of the file:
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@@
-		)
-	)
-	(label "SYNC"
-		(at 146.05 182.88 270)
-		(fields_autoplaced yes)
-		(effects
-			(font
-				(size 1.27 1.27)
-			)
-			(justify right bottom)
 		)
 	)
