File: ch32m030/fets.kicad_sch (KiCad schematic)
At the start: 81 parts, among them Q1 BSC019N06NSATMA1, Q2 BSC019N06NSATMA1, Q3 BSC019N06NSATMA1, Q4 BSC019N06NSATMA1, Q5 BSC019N06NSATMA1, Q6 BSC019N06NSATMA1, Q7 BSC019N06NSATMA1, Q8 BSC019N06NSATMA1

Commit message: v1
Connections:
- net GNDPWR is gone; now on net GND: C12.2, C13.2, C18.2, C19.2, C24.2, C25.2, C6.2, C7.2, R19.2, R20.2, R57.2, R59.2, R7.2, R8.2
Other:
- note added: "IAUC120N06S5L011ATMA1"

Commit message: add ch32v307drv
Parts:
- removed C10, C11, C16, C17, C22, C23, C4, C5: 1uF, PCM_JLCPCB:C_0603, symbol PCM_JLCPCB-Capacitors:0603,1uF
