File: ch32v307drv/ch32v307drv.kicad_pcb (KiCad board)
At the start: 4 copper layers, 65.5 x 100.3 mm, 138 parts, among them J1 TBL002A-350-10GY-2GY, J2 Connector, USB-TYPE-C-16P, J3 691256610006, J4 SM06B-SRSS-TBLFSN, P1 2204061-2 Edge Connector, Q1 BSC019N06NSATMA1, Q2 BSC019N06NSATMA1, Q3 BSC019N06NSATMA1, Q4 BSC019N06NSATMA1, Q5 BSC019N06NSATMA1, Q6 BSC019N06NSATMA1, Q7 BSC019N06NSATMA1, Q8 BSC019N06NSATMA1, U1 CH32M030C8U3, U2 HT7533, U3 CH221K, X1 X50328MSB2GI

Commit message: more design
Parts:
- removed C1, C2, C41: 10uF, PCM_JLCPCB:C_1206
- removed C26, C27: 2.2uF, PCM_JLCPCB:C_1206
- removed C28, C29, C30, C31: 10nF, PCM_JLCPCB:C_0603
- removed C40: 1uF, PCM_JLCPCB:C_0603
- removed C42: 100nF, PCM_JLCPCB:C_0603
- removed D7: SRV05-4_C7420376, PCM_JLCPCB:SOT-23-6_L2.9-W1.6-P0.95-LS2.8-BL-1
- removed JP1, JP2, JP3, JP4, JP5, JP6, JP7, JP8: SolderJumper_2_Open, Jumper:SolderJumper-2_P1.3mm_Open_TrianglePad1.0x1.5mm
- removed P1: 2204061-2 Edge Connector, 2204061-2_edge:edge
- removed Q1, Q2, Q3, Q4, Q5, Q6, Q7, Q8: BSC019N06NSATMA1, Package_SON:Infineon_PG-TDSON-8_6.15x5.15mm
- removed R33, R34, R35, R36, R37, R38, R39, R40: 1.5kΩ, PCM_JLCPCB:R_0603
- removed R41: 100kΩ, PCM_JLCPCB:R_0603
- removed R42: 6.2kΩ, PCM_JLCPCB:R_0603
- removed R43: 200kΩ, PCM_JLCPCB:R_0603
- removed R44: 1kΩ, PCM_JLCPCB:R_0603
- removed R47, R48, R49, R51, R52, R53, R54: 33Ω, PCM_JLCPCB:R_0603
- removed R50: 10Ω, PCM_JLCPCB:R_0603
- removed R56, R57, R58, R59: 0Ω, PCM_JLCPCB:R_0603
- removed R61: 10kΩ, PCM_JLCPCB:R_0603
- added C43: 10nF, PCM_JLCPCB:C_0603, F.Cu at (96.5, 108.7)
- added C44: 10nF, PCM_JLCPCB:C_0603, F.Cu at (96.5, 110.9)
- added C47: 100nF, PCM_JLCPCB:C_0603, F.Cu at (96.5, 113.2)
- added C48: 100nF, PCM_JLCPCB:C_0603, F.Cu at (96.5, 115.4)
- added C50: 100nF, PCM_JLCPCB:C_1206, F.Cu at (74.3, 95.8)
- added C51: 100nF, PCM_JLCPCB:C_1206, F.Cu at (74.3, 99.2)
- added C52: 330pF, PCM_JLCPCB:C_1206, F.Cu at (69.2, 95.7)
- added C53: 330pF, PCM_JLCPCB:C_1206, F.Cu at (244.0, 125.2)
- added C54: 100nF, PCM_JLCPCB:C_1206, F.Cu at (74.3, 102.5)
- added C55: 100nF, PCM_JLCPCB:C_0603, F.Cu at (96.5, 117.7)
- added C56: 100nF, PCM_JLCPCB:C_0603, F.Cu at (100.4, 108.7)
- added C57: 100nF, PCM_JLCPCB:C_0603, F.Cu at (100.4, 110.9)
- added C58: 100nF, PCM_JLCPCB:C_0603, F.Cu at (100.4, 113.2)
- added C59: 100nF, PCM_JLCPCB:C_0603, F.Cu at (100.4, 115.4)
- added C60: 100nF, PCM_JLCPCB:C_1206, F.Cu at (74.3, 105.8)
- added C62: 100nF, PCM_JLCPCB:C_1206, F.Cu at (79.9, 95.8)
- added C63: 100nF, PCM_JLCPCB:C_1206, F.Cu at (79.9, 99.2)
- added C64: 100nF, PCM_JLCPCB:C_0603, F.Cu at (100.4, 117.7)
- added C65: 330pF, PCM_JLCPCB:C_1206, F.Cu at (69.2, 101.8)
- added C66: 330pF, PCM_JLCPCB:C_1206, F.Cu at (269.6, 125.2)
- added C67: 100nF, PCM_JLCPCB:C_0603, F.Cu at (126.2, 76.2)
- added C68: 100nF, PCM_JLCPCB:C_0603, F.Cu at (126.2, 78.5)
- added C69: 100nF, PCM_JLCPCB:C_1206, F.Cu at (79.9, 102.5)
- added C71: 100nF, PCM_JLCPCB:C_1206, F.Cu at (79.9, 105.8)
- added C72: 100nF, PCM_JLCPCB:C_1206, F.Cu at (85.6, 95.8)
- added C73: 100nF, PCM_JLCPCB:C_0603, F.Cu at (126.2, 80.8)
- added C74: 330pF, PCM_JLCPCB:C_1206, F.Cu at (69.2, 107.8)
- added C75: 330pF, PCM_JLCPCB:C_1206, F.Cu at (256.8, 125.0)
- added C76: 100nF, PCM_JLCPCB:C_0603, F.Cu at (126.2, 83.0)
- added C77: 100nF, PCM_JLCPCB:C_1206, F.Cu at (85.6, 99.2)
- added C79: 100nF, PCM_JLCPCB:C_1206, F.Cu at (85.6, 102.5)
- added C80: 100nF, PCM_JLCPCB:C_1206, F.Cu at (85.6, 105.8)
- added C81: 330pF, PCM_JLCPCB:C_1206, F.Cu at (69.2, 114.0)
- added C82: 330pF, PCM_JLCPCB:C_1206, F.Cu at (281.2, 125.2)
- added D10: SRV05-4_C7420376, PCM_JLCPCB:SOT-23-6_L2.9-W1.6-P0.95-LS2.8-BL-1, F.Cu at (46.7, 48.0)
- added D11: SRV05-4_C7420376, PCM_JLCPCB:SOT-23-6_L2.9-W1.6-P0.95-LS2.8-BL-1, F.Cu at (50.8, 48.0)
- added D12: H3V3HT2B, PCM_JLCPCB:SOT-23-3_L2.9-W1.3-P1.90-LS2.4-BR, F.Cu at (72.8, 58.4)
- added D13: H3V3HT2B, PCM_JLCPCB:SOT-23-3_L2.9-W1.3-P1.90-LS2.4-BR, F.Cu at (39.5, 52.8)
- added D14: SRV05-4_C7420376, PCM_JLCPCB:SOT-23-6_L2.9-W1.6-P0.95-LS2.8-BL-1, F.Cu at (130.2, 72.9)
- added D15: SS220, PCM_JLCPCB:D_SMA, F.Cu at (114.7, 79.7)
- added D9: BZT52C3V9S, PCM_JLCPCB:D_SOD-323, F.Cu at (55.0, 157.4)
- added J5: RJ45_Hanrun_HR911105A_Horizontal, Connector_RJ:RJ45_Hanrun_HR911105A_Horizontal, F.Cu at (215.5, 68.8)
- added J6: 691256610006, 691256610006 (1):691256610006, F.Cu at (265.7, 133.9)
- added J7: SS-6466S-A-PG1, SS_6466S_A_PG1:BEL_SS-6466S-A-PG1, F.Cu at (208.8, 54.9)
- added L1: XGL1010-122MED, Inductor_SMD:L_Coilcraft_XAL1010-XXX, F.Cu at (263.2, 117.8)
- added L2: XGL1010-122MED, Inductor_SMD:L_Coilcraft_XAL1010-XXX, F.Cu at (275.8, 117.7)
- added L3: XGL1010-122MED, Inductor_SMD:L_Coilcraft_XAL1010-XXX, F.Cu at (250.6, 117.8)
- added L4: XGL4040-223MEC, Inductor_SMD:L_Coilcraft_XAL4040-XXX, F.Cu at (119.3, 84.9)
- added L5: XGL1010-122MED, Inductor_SMD:L_Coilcraft_XAL1010-XXX, F.Cu at (237.8, 117.8)
- added R100: 10kΩ, PCM_JLCPCB:R_0603, F.Cu at (80.6, 117.7)
- added R101: 10kΩ, PCM_JLCPCB:R_0603, F.Cu at (80.6, 119.9)
- added R102: 10kΩ, PCM_JLCPCB:R_0603, F.Cu at (84.2, 108.7)
- added R103: 10kΩ, PCM_JLCPCB:R_0603, F.Cu at (84.2, 110.9)
- added R104: 10kΩ, PCM_JLCPCB:R_0603, F.Cu at (84.2, 113.2)
- added R105: 2Ohm 0805 Thick FIlm Resistor, Resistor_SMD:R_0805_2012Metric, F.Cu at (88.2, 125.2)
- added R106: 2Ohm 0805 Thick FIlm Resistor, Resistor_SMD:R_0805_2012Metric, F.Cu at (88.2, 128.2)
- added R107: 2Ohm 0805 Thick FIlm Resistor, Resistor_SMD:R_0805_2012Metric, F.Cu at (88.2, 131.1)
- added R108: 47kΩ, PCM_JLCPCB:R_0603, F.Cu at (84.2, 115.4)
- added R72: 220Ω, PCM_JLCPCB:R_0603, F.Cu at (54.6, 143.6)
- added R73: 220Ω, PCM_JLCPCB:R_0603, F.Cu at (54.6, 145.8)
- added R74: 0Ω, PCM_JLCPCB:R_0603, F.Cu at (54.6, 148.1)
- added R75: 0Ω, PCM_JLCPCB:R_0603, F.Cu at (54.6, 150.3)
- added R76: 0Ω, PCM_JLCPCB:R_0603, F.Cu at (54.6, 152.6)
- added R77: 0Ω, PCM_JLCPCB:R_0603, F.Cu at (54.6, 154.8)
- added R78: 47kΩ, PCM_JLCPCB:R_0603, F.Cu at (73.3, 108.7)
- added R79: 47kΩ, PCM_JLCPCB:R_0603, F.Cu at (73.3, 110.9)
- added R80: 47kΩ, PCM_JLCPCB:R_0603, F.Cu at (73.3, 113.2)
- added R82: 1.5kΩ, PCM_JLCPCB:R_0603, F.Cu at (73.3, 115.4)
- added R84: 1.5kΩ, PCM_JLCPCB:R_0603, F.Cu at (73.3, 117.7)
- added R86: 1.5kΩ, PCM_JLCPCB:R_0603, F.Cu at (73.3, 119.9)
- added R87: 1.5kΩ, PCM_JLCPCB:R_0603, F.Cu at (76.9, 108.7)
- added R88: 1.5kΩ, PCM_JLCPCB:R_0603, F.Cu at (76.9, 110.9)
- added R89: 1.5kΩ, PCM_JLCPCB:R_0603, F.Cu at (76.9, 113.2)
- added R90: 1.5kΩ, PCM_JLCPCB:R_0603, F.Cu at (76.9, 115.4)
- added R91: 1.5kΩ, PCM_JLCPCB:R_0603, F.Cu at (76.9, 117.7)
- added R94: 2Ohm 0805 Thick FIlm Resistor, Resistor_SMD:R_0805_2012Metric, F.Cu at (88.2, 122.3)
- added R95: 10kΩ, PCM_JLCPCB:R_0603, F.Cu at (76.9, 119.9)
- added R96: 10kΩ, PCM_JLCPCB:R_0603, F.Cu at (80.6, 108.7)
- added R97: 10kΩ, PCM_JLCPCB:R_0603, F.Cu at (80.6, 110.9)
- added R98: 10kΩ, PCM_JLCPCB:R_0603, F.Cu at (80.6, 113.2)
- added R99: 10kΩ, PCM_JLCPCB:R_0603, F.Cu at (80.6, 115.4)
- added U12: LMG2100R026VBNR, lmg2100:VBN0018A-MFG, B.Cu at (264.1, 106.6)
- added U13: SN74LVC7001ABQAR, sn74:PW14, F.Cu at (75.9, 124.4)
- added U14: SN74LVC7001ABQAR, sn74:PW14, F.Cu at (75.9, 131.2)
- added U15: ACS37032LLZATR-065B3, acs3703:SOIC6_LZ_ALM, F.Cu at (235.2, 109.1)
- added U16: LMG2100R026VBNR, lmg2100:VBN0018A-MFG, B.Cu at (257.1, 106.6)
- added U17: ACS37032LLZATR-065B3, acs3703:SOIC6_LZ_ALM, F.Cu at (260.6, 109.1)
- added U18: LMG2100R026VBNR, lmg2100:VBN0018A-MFG, B.Cu at (250.2, 106.6)
- added U19: LMG2100R026VBNR, lmg2100:VBN0018A-MFG, B.Cu at (243.2, 106.6)
- added U4: SN65HVD230DR, PCM_JLCPCB:SOIC-8_L4.9-W3.9-P1.27-LS6.0-BL, F.Cu at (67.6, 56.1)
- added U5: LTV-827S, Package_DIP:SMDIP-8_W9.53mm, F.Cu at (71.1, 39.4)
- added U6: LM5012DDAR, lmg5012:DDA0008E-MFG, F.Cu at (116.0, 74.0)
- added U7: LTV-827S, Package_DIP:SMDIP-8_W9.53mm, F.Cu at (120.7, 46.9)
- C10, C11: footprint PCM_JLCPCB:C_0603 -> PCM_JLCPCB:C_1206
- C12: value 100uF 50V C311622 -> 1uF; footprint Capacitor_SMD:CP_Elec_6.3x7.7 -> PCM_JLCPCB:C_1206
- C13, C32: value 10uF -> 100nF
- C14: value 2.2uF -> 1uF; footprint PCM_JLCPCB:C_1206 -> PCM_JLCPCB:C_0603
- C15: value 2.2uF -> 100nF
- C16, C3, C4: value 1uF -> 100nF
- C17, C22: value 1uF -> 100nF; footprint PCM_JLCPCB:C_0603 -> PCM_JLCPCB:C_1206
- C18: value 100uF 50V C311622 -> 100nF; footprint Capacitor_SMD:CP_Elec_6.3x7.7 -> PCM_JLCPCB:C_0603
- C19: footprint PCM_JLCPCB:C_1206 -> PCM_JLCPCB:C_0603
- C20: value 2.2uF -> 10uF; footprint PCM_JLCPCB:C_1206 -> PCM_JLCPCB:C_0603
- C21, C9: value 2.2uF -> 1uF
- C23: value 1uF -> 2.2nF
- C24: value 100uF 50V C311622 -> 2.2nF; footprint Capacitor_SMD:CP_Elec_6.3x7.7 -> PCM_JLCPCB:C_0603
- C25: value 10uF -> 100nF; footprint PCM_JLCPCB:C_1206 -> PCM_JLCPCB:C_0603
- C33: value 10uF -> 1uF; footprint PCM_JLCPCB:C_1206 -> PCM_JLCPCB:C_0603
- C34, C35: value 10uF -> 10nF; footprint PCM_JLCPCB:C_1206 -> PCM_JLCPCB:C_0603
- C5: value 1uF -> 10uF
- C6: value 100uF 50V C311622 -> 10uF; footprint Capacitor_SMD:CP_Elec_6.3x7.7 -> PCM_JLCPCB:C_0603
- C7: value 10uF -> 22uF 100V C88689; footprint PCM_JLCPCB:C_1206 -> Capacitor_SMD:CP_Elec_10x10
- C8: value 2.2uF -> 22uF 100V C88689; footprint PCM_JLCPCB:C_1206 -> Capacitor_SMD:CP_Elec_10x10
- D2: value SK1010C -> 1N4004W; footprint PCM_JLCPCB:D_SMC -> PCM_JLCPCB:D_SOD-123FL
- D8: value SRV05-4_C7420376 -> BZT52C3V9S; footprint PCM_JLCPCB:SOT-23-6_L2.9-W1.6-P0.95-LS2.8-BL-1 -> PCM_JLCPCB:D_SOD-323
- J1: value TBL002A-350-10GY-2GY -> SS-641010S-A-NF; footprint TBL002A_350_10GY_2GY (1):CUI_TBL002A-350-10GY-2GY -> SS_641010S_A_NF:BEL_SS-641010S-A-NF
- J3: value 691256610006 -> SS-6466S-A-PG1; footprint 691256610006 (1):691256610006 -> SS_6466S_A_PG1:BEL_SS-6466S-A-PG1
- R1, R15, R2: value 10Ω -> 10kΩ
- R10: value 10Ω -> 1.5kΩ
- R11: value 10kΩ -> 1.5kΩ
- R12: value 10kΩ -> 1kΩ
- R13, R14, R27: value 2Ω -> 1kΩ
- R16: value 10Ω -> 33Ω
- R17, R18: value 10kΩ -> 33Ω
- R19, R20: value 0.005Ohm C2994643 -> 33Ω; footprint Resistor_SMD:R_2512_6332Metric -> PCM_JLCPCB:R_0603
- R21: value 2Ω -> 33Ω
- R22: value 2Ω -> 120Ω
- R23, R24: value 10Ω -> 330Ω
- R25: value 10kΩ -> 15kΩ
- R26: value 10kΩ -> 100kΩ
- R28: value 2Ω -> 30kΩ
- R29: value 10kΩ -> 100kΩ; moved to F.Cu
- R30: value 10kΩ -> 30kΩ; moved to F.Cu
- R31, R32: value 10kΩ -> 330Ω; moved to F.Cu
- R5, R6: value 2Ω -> 100kΩ
- R7, R8: value 0.005Ohm C2994643 -> 100kΩ; footprint Resistor_SMD:R_2512_6332Metric -> PCM_JLCPCB:R_0603
- R9: value 10Ω -> 47kΩ
- U1: value CH32M030C8U3 -> CH32V30xVxTx; footprint Package_DFN_QFN:QFN-48-1EP_7x7mm_P0.5mm_EP3.5x3.5mm -> Package_QFP:LQFP-100_14x14mm_P0.5mm
- U2: value HT7533 -> AMS1117; footprint PCM_JLCPCB:SOT-89-3_L4.5-W2.5-P1.50-LS4.2-BR -> PCM_JLCPCB:SOT-223-3_L6.5-W3.4-P2.30-LS7.0-BR
- U3: value CH221K -> AM26LV32xD; footprint CH221K:SOT95P280X120-6N -> Package_SO:SOIC-16_3.9x9.9mm_P1.27mm
- moved C7 150.9 mm to (289.0, 107.2), turned to 180 degrees
- moved R20 147.3 mm to (39.2, 45.4)
- moved R19 146.2 mm to (39.2, 43.1)
- moved C8 145.1 mm to (289.0, 119.0), turned to 180 degrees
- moved R18 140.9 mm to (39.2, 40.9)
- moved R16 140.7 mm to (39.2, 36.4)
- moved J2 140.7 mm to (278.1, 51.1)
- moved R14 136.3 mm to (39.2, 34.1)
- moved J1 134.2 mm to (224.2, 134.8), turned to 0 degrees
- moved R17 132.5 mm to (39.2, 38.6)
- moved C9 129.9 mm to (26.3, 96.2)
- moved C11 129.7 mm to (26.3, 102.8)
- moved R13 128.4 mm to (39.2, 31.9)
- moved J4 128.1 mm to (289.3, 48.9)
- moved R21 126.8 mm to (39.2, 47.6)
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Connections:
- C10 pad 1: Net-(Q3-G) -> VBUS
- C10 pad 2: /SW1 -> GND
- C11 pad 1: Net-(Q4-G) -> VBUS
- C11 pad 2: Net-(C11-Pad2) -> GND
- C12 pad 1: +24V -> VBUS
- C13 pad 1: +24V -> Net-(J1-SHIELD)
- C14 pad 1: Net-(C14-Pad1) -> GND
- C14 pad 2: /SW1 -> +3V3
- C15 pad 1: Net-(C15-Pad1) -> Net-(J3-SHIELD)
- C15 pad 2: Net-(C11-Pad2) -> GND
- C16 pad 1: Net-(Q5-G) -> GND
- C16 pad 2: /SW2 -> +3V3
- C17 pad 1: Net-(Q6-G) -> Net-(J7-SHIELD)
- C17 pad 2: Net-(C17-Pad2) -> GND
- C18 pad 1: +24V -> +5V
- C19 pad 1: +24V -> +5V
- C20 pad 1: Net-(C20-Pad1) -> +5V
- C20 pad 2: /SW2 -> GND
- C21 pad 1: Net-(C21-Pad1) -> GND
- C21 pad 2: Net-(C17-Pad2) -> VBUS
- C22 pad 1: Net-(Q7-G) -> GND
- C22 pad 2: /SW3 -> VBUS
- C23 pad 1: Net-(Q8-G) -> Net-(U6-BST)
- C23 pad 2: Net-(C17-Pad2) -> Net-(U6-SW)
- C24 pad 1: +24V -> Net-(C24-Pad1)
- C24 pad 2: GND -> +5V
- C25 pad 1: +24V -> Net-(C24-Pad1)
- C25 pad 2: GND -> Net-(U6-FB)
- C32 pad 1: Net-(U1-VBOOT3) -> Net-(C32-Pad1)
- C32 pad 2: /SW3 -> GND
- C33 pad 1: Net-(U1-VBOOT2) -> +3V3
- C33 pad 2: /SW2 -> GND
- C34 pad 1: Net-(U1-VBOOT1) -> GND
- C34 pad 2: /SW1 -> /BEMF_U
- C35 pad 1: Net-(U1-VBOOT0) -> GND
- C35 pad 2: /SW0 -> /BEMF_V
- C37 pad 2: Net-(U1-PB4/V_DET/A17) -> /VBUS_MON
- C38 pad 2: Net-(U1-PB5/XI/CM2P/A3) -> Net-(U1-OSC_IN)
- C39 pad 2: Net-(U1-PB6/X0/CM2N/A4) -> Net-(U1-OSC_OUT)
- C4 pad 1: Net-(Q1-G) -> GND
- C4 pad 2: /SW0 -> /VGG_MON
- C5 pad 1: Net-(Q2-G) -> +5V
- C5 pad 2: Net-(C11-Pad2) -> GND
- C6 pad 1: +24V -> +3V3
- C7 pad 1: +24V -> VBUS
- C8 pad 1: Net-(C8-Pad1) -> VBUS
- C8 pad 2: /SW0 -> GND
- C9 pad 1: Net-(C9-Pad1) -> VBUS
- C9 pad 2: Net-(C11-Pad2) -> GND
- D2 pad 1: +24V -> +5V
- D6 pad 3: /SYNC -> unconnected-(D6-I/O-Pad3)
- D8 pad 1: /BEMF_W -> /VBUS_MON
- J1 pad 1: Net-(J1-Pad1) -> GND
- J1 pad 10: /HV_IO -> /encoder1/DIFF_REF
- J1 pad 2: Net-(J1-Pad2) -> /encoder1/AP
- J1 pad 3: Net-(J1-Pad3) -> /encoder1/AN
- J1 pad 4: Net-(J1-Pad4) -> /encoder1/BP
- J1 pad 5: Net-(J1-Pad5) -> /encoder1/BN
- J1 pad 6: Net-(J1-Pad6) -> /encoder1/ZP
- J1 pad 7: Net-(J1-Pad7) -> /encoder1/ZN
- J1 pad 8: Net-(J1-Pad8) -> +5V
- J1 pad 9: GND -> +3V3
- J3 pad 1: /SW0 -> Net-(U4-VREF)
- J3 pad 2: /SW1 -> GND
- J3 pad 3: /SW2 -> Net-(U4-CANL)
- J3 pad 4: /SW3 -> Net-(U4-CANH)
- J3 pad 5: +24V -> GND
- J3 pad 6: GND -> Net-(U4-RS)
- R1 pad 1: /fets/VGH0 -> /BEMF_U
- R1 pad 2: Net-(Q1-G) -> Net-(U1-PB15)
- R10 pad 1: /fets/VGL1 -> /VBUS_MON
- R10 pad 2: Net-(Q4-G) -> GND
- R11 pad 1: Net-(Q3-G) -> /VGG_MON
- R11 pad 2: /SW1 -> GND
- R12 pad 1: Net-(Q4-G) -> +5V
- R12 pad 2: Net-(C11-Pad2) -> /VGG_MON
- R13 pad 1: +24V -> /encoder1/DIFF_REF
- R13 pad 2: Net-(C14-Pad1) -> +3V3
- R14 pad 1: /SW1 -> GND
- R14 pad 2: Net-(C15-Pad1) -> /encoder1/DIFF_REF
- R15 pad 1: /fets/VGH2 -> Net-(U4-RS)
- R15 pad 2: Net-(Q5-G) -> +3V3
- R16 pad 1: /fets/VGL2 -> /encoder1/AP
- R16 pad 2: Net-(Q6-G) -> Net-(U3-1A)
- R17 pad 1: Net-(Q5-G) -> /encoder1/AN
- R17 pad 2: /SW2 -> Net-(U3-1B)
- R18 pad 1: Net-(Q6-G) -> /encoder1/BP
- R18 pad 2: Net-(C17-Pad2) -> Net-(U3-2A)
- R19 pad 1: Net-(C17-Pad2) -> /encoder1/BN
- R19 pad 2: GND -> Net-(U3-2B)
- R2 pad 1: /fets/VGL0 -> /BEMF_V
- R2 pad 2: Net-(Q2-G) -> Net-(U1-PB14)
- R20 pad 1: Net-(C17-Pad2) -> /encoder1/ZP
- R20 pad 2: GND -> Net-(U3-3A)
- R21 pad 1: +24V -> /encoder1/ZN
- R21 pad 2: Net-(C20-Pad1) -> Net-(U3-3B)
- R22 pad 1: /SW2 -> Net-(U4-CANL)
- R22 pad 2: Net-(C21-Pad1) -> Net-(U4-CANH)
- R23 pad 1: /fets/VGH3 -> Net-(R23-Pad1)
- R23 pad 2: Net-(Q7-G) -> Net-(J7-Pad2)
- R24 pad 1: /fets/VGL3 -> Net-(R24-Pad1)
- R24 pad 2: Net-(Q8-G) -> Net-(J7-Pad3)
- R25 pad 1: Net-(Q7-G) -> Net-(U6-RON)
- R25 pad 2: /SW3 -> GND
- R26 pad 1: Net-(Q8-G) -> +5V
- R26 pad 2: Net-(C17-Pad2) -> Net-(U6-FB)
- R27 pad 1: +24V -> Net-(R27-Pad1)
- R27 pad 2: Net-(C26-Pad1) -> GND
- R28 pad 1: /SW3 -> Net-(U6-FB)
- R28 pad 2: Net-(C27-Pad1) -> Net-(R27-Pad1)
- R29 pad 1: /SW0 -> Net-(U6-SW)
- R29 pad 2: /BEMF_U -> Net-(R29-Pad2)
- R3 pad 1: Net-(Q1-G) -> /BEMF_W
- R3 pad 2: /SW0 -> Net-(U1-PB13)
- R30 pad 1: /SW1 -> Net-(R29-Pad2)
- R30 pad 2: /BEMF_V -> Net-(C24-Pad1)
- R31 pad 1: /SW2 -> Net-(R31-Pad1)
- R31 pad 2: /BEMF_W -> Net-(J7-Pad5)
- R32 pad 1: /SW3 -> Net-(R32-Pad1)
- R32 pad 2: /BEMF_X -> Net-(J7-Pad6)
- R4 pad 1: Net-(Q2-G) -> /BEMF_X
- R4 pad 2: Net-(C11-Pad2) -> Net-(U1-PB12)
- R5 pad 1: +24V -> /OPA_O_U
- R5 pad 2: Net-(C8-Pad1) -> Net-(U1-PB15)
- R6 pad 1: /SW0 -> /OPA_O_V
- R6 pad 2: Net-(C9-Pad1) -> Net-(U1-PB14)
- R7 pad 1: Net-(C11-Pad2) -> /OPA_O_W
- R7 pad 2: GND -> Net-(U1-PB13)
- R8 pad 1: Net-(C11-Pad2) -> /OPA_O_X
- R8 pad 2: GND -> Net-(U1-PB12)
- R9 pad 1: /fets/VGH1 -> /VBUS_MON
- R9 pad 2: Net-(Q3-G) -> VBUS
- U1 pad 1: /IS_2_P -> unconnected-(U1-PE2-Pad1)
- U1 pad 10: Net-(U1-PB5/XI/CM2P/A3) -> GND
- U1 pad 11: Net-(U1-PB6/X0/CM2N/A4) -> +3V3
- U1 pad 12: /fets/VGL0 -> Net-(U1-OSC_IN)
- U1 pad 13: /SW0 -> Net-(U1-OSC_OUT)
- U1 pad 14: Net-(U1-VBOOT0) -> /RST
- U1 pad 15: /fets/VGH0 -> /VGG_MON
- U1 pad 16: /fets/VGL1 -> /VBUS_MON
- U1 pad 17: /SW1 -> unconnected-(U1-PC2-Pad17)
- U1 pad 18: Net-(U1-VBOOT1) -> unconnected-(U1-PC3-Pad18)
- U1 pad 19: /fets/VGH1 -> GND
- U1 pad 2: /IS_2_N -> unconnected-(U1-PE3-Pad2)
- U1 pad 20: /fets/VGL2 -> unconnected-(U1-VREF--Pad20)
- U1 pad 21: /SW2 -> unconnected-(U1-VREF+-Pad21)
- U1 pad 22: Net-(U1-VBOOT2) -> +3V3
- U1 pad 23: /fets/VGH2 -> /OPA_O_X
- U1 pad 24: /fets/VGL3 -> /OPA_O_W
- U1 pad 25: /SW3 -> /OPA_O_V
- U1 pad 26: Net-(U1-VBOOT3) -> /OPA_O_U
- U1 pad 27: /fets/VGH3 -> GND
- U1 pad 28: +12V -> +3V3
- U1 pad 29: /HV_TACH -> unconnected-(U1-PA4-Pad29)
- U1 pad 3: /LIM_L -> /ENC0_A
- U1 pad 30: /UART_RX -> unconnected-(U1-PA5-Pad30)
- U1 pad 31: /UART_TX -> /U_I
- U1 pad 32: /SPI_MOSI -> /U_I
- U1 pad 33: /SPI_MISO -> unconnected-(U1-PC4-Pad33)
- U1 pad 34: /HV_IO -> unconnected-(U1-PC5-Pad34)
- U1 pad 35: +3V3 -> /PWML3
- U1 pad 36: +24V -> /BEMF_C
- U1 pad 37: /SPI_NSS -> /BEMF_C
- U1 pad 38: /SPI_SCK -> unconnected-(U1-PE7-Pad38)
- U1 pad 39: /SWCLK -> /PWML0
- U1 pad 4: /BRAKE -> /ENC0_B
- U1 pad 40: /SWIO -> unconnected-(U1-PE9-Pad40)
- U1 pad 41: /USBFS_P -> /PWML1
- U1 pad 42: /USBFS_N -> unconnected-(U1-PE11-Pad42)
- U1 pad 43: /SYNC -> /PWML2
- U1 pad 44: /BEMF_U -> /LIM_L
- U1 pad 45: /BEMF_V -> /LIM_H
- U1 pad 46: /BEMF_W -> /STO_H
- U1 pad 47: /IS_1_N -> /BEMF_C
- U1 pad 48: /IS_1_P -> /BEMF_C
- U1 pad 5: /LIM_H -> /ENC0_C
- U1 pad 6: /RST -> unconnected-(U1-VBAT-Pad6)
- U1 pad 7: /BEMF_X -> unconnected-(U1-PC13-Pad7)
- U1 pad 8: /BEMF_C -> unconnected-(U1-PC14-Pad8)
- U1 pad 9: Net-(U1-PB4/V_DET/A17) -> unconnected-(U1-PC15-Pad9)
- U2 pad 2: Net-(JP8-B) -> +3V3
- U2 pad 3: +3V3 -> +5V
- U3 pad 1: Net-(U3-VDD) -> Net-(U3-1B)
- U3 pad 2: GND -> Net-(U3-1A)
- U3 pad 3: /USB_PD_ACTIVE -> /ENC0_A
- U3 pad 4: Net-(J2-CC1) -> +3V3
- U3 pad 5: Net-(J2-CC2) -> /ENC0_B
- U3 pad 6: Net-(U3-CFG) -> Net-(U3-2A)
- X1 pad 1: Net-(U1-PB6/X0/CM2N/A4) -> Net-(U1-OSC_OUT)
- X1 pad 2: Net-(U1-PB5/XI/CM2P/A3) -> Net-(U1-OSC_IN)
Routing:
- removed copper zone on B.Cu, net +24V
- removed copper zone on F.Cu, net +24V
- removed copper zone on In1.Cu, net +24V
- removed copper zone on In2.Cu, net +24V
- removed copper zone on In2.Cu, net +3V3
- removed copper zone on B.Cu, net /SW0
- removed copper zone on F.Cu, net /SW0
- removed copper zone on In1.Cu, net /SW0
- removed copper zone on In2.Cu, net /SW0
- removed copper zone on B.Cu, net /SW1
- removed copper zone on F.Cu, net /SW1
- removed copper zone on In1.Cu, net /SW1
- removed copper zone on In2.Cu, net /SW1
- removed copper zone on B.Cu, net /SW2
- removed copper zone on F.Cu, net /SW2
- removed copper zone on In1.Cu, net /SW2
- removed copper zone on In2.Cu, net /SW2
- removed copper zone on B.Cu, net /SW3
- removed copper zone on F.Cu, net /SW3
- removed copper zone on In1.Cu, net /SW3
- removed copper zone on In2.Cu, net /SW3
- removed copper zone on B.Cu, net GND
- removed copper zone on F.Cu, net GND
- removed copper zone on In1.Cu, net GND
- removed copper zone on In2.Cu, net GND
- removed copper zone on F.Cu, net Net-(C11-Pad2)
- removed copper zone on In1.Cu, net Net-(C11-Pad2)
- removed copper zone on F.Cu, net Net-(C17-Pad2)
- removed copper zone on In1.Cu, net Net-(C17-Pad2)
Other:
- board size 65.5 x 100.3 mm -> 101.8 x 101.8 mm
- board text removed: "EXT 3v3"
