File: ch32v307drv/ch32v307drv.kicad_sch (KiCad schematic)
At the start: 45 parts, among them J1 TBL002A-350-10GY-2GY, J4 SM06B-SRSS-TBLFSN, J5 RJ45_Hanrun_HR911105A_Horizon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, U1 CH32V30xVxTx, U2 HT7533, X1 X50328MSB2GI

Commit message: more design
Parts:
- removed C1, C2, C41: 10uF, PCM_JLCPCB:C_1206, symbol PCM_JLCPCB-Capacitors:1206,10uF
- removed C3: 1uF, PCM_JLCPCB:C_0603, symbol PCM_JLCPCB-Capacitors:0603,1uF
- removed C42: 100nF, PCM_JLCPCB:C_0603, symbol PCM_JLCPCB-Capacitors:0603,100nF
- removed D7: SRV05-4_C7420376, PCM_JLCPCB:SOT-23-6_L2.9-W1.6-P0.95-LS2.8-BL-1, symbol PCM_JLCPCB-Diode-Packages:Package, SRV05-4_C7420376
- removed J1: TBL002A-350-10GY-2GY, TBL002A_350_10GY_2GY (1):CUI_TBL002A-350-10GY-2GY, symbol TBL002A-350-10GY-2GY:TBL002A-350-10GY-2GY
- removed JP8: SolderJumper_2_Open, Jumper:SolderJumper-2_P1.3mm_Open_TrianglePad1.0x1.5mm, symbol Jumper:SolderJumper_2_Open
- removed R41: 100kΩ, PCM_JLCPCB:R_0603, symbol PCM_JLCPCB-Resistors:0603,100kΩ
- removed R42: 6.2kΩ, PCM_JLCPCB:R_0603, symbol PCM_JLCPCB-Resistors:0603,6.2kΩ
- removed R47, R48, R49, R51, R52, R53, R54: 33Ω, PCM_JLCPCB:R_0603, symbol PCM_JLCPCB-Resistors:0603,33Ω
- removed R50: 10Ω, PCM_JLCPCB:R_0603, symbol PCM_JLCPCB-Resistors:0603,10Ω
- removed R61: 10kΩ, PCM_JLCPCB:R_0603, symbol PCM_JLCPCB-Resistors:0603,10kΩ
- removed U2: HT7533, PCM_JLCPCB:SOT-89-3_L4.5-W2.5-P1.50-LS4.2-BR, symbol PCM_JLCPCB-Power:LDO, 3.3V, 0.1A
- added C17: 100nF, PCM_JLCPCB:C_1206, symbol PCM_JLCPCB-Capacitors:1206,100nF
- added C3, C4: 100nF, PCM_JLCPCB:C_0603, symbol PCM_JLCPCB-Capacitors:0603,100nF
- added C5, C6: 10uF, PCM_JLCPCB:C_0603, symbol PCM_JLCPCB-Capacitors:0603,10uF
- added D8, D9: BZT52C3V9S, PCM_JLCPCB:D_SOD-323, symbol PCM_JLCPCB-Diodes:Zener,BZT52C3V9S
- added J7: SS-6466S-A-PG1, SS_6466S_A_PG1:BEL_SS-6466S-A-PG1, symbol SS-6466S-A-PG1:SS-6466S-A-PG1
- added R1, R2, R3, R4: 10kΩ, PCM_JLCPCB:R_0603, symbol PCM_JLCPCB-Resistors:0603,10kΩ
- added R10, R11: 1.5kΩ, PCM_JLCPCB:R_0603, symbol PCM_JLCPCB-Resistors:0603,1.5kΩ
- added R12: 1kΩ, PCM_JLCPCB:R_0603, symbol PCM_JLCPCB-Resistors:0603,1kΩ
- added R23, R24, R31, R32: 330Ω, PCM_JLCPCB:R_0603, symbol PCM_JLCPCB-Resistors:0603,330Ω
- added R5, R6, R7, R8: 100kΩ, PCM_JLCPCB:R_0603, symbol PCM_JLCPCB-Resistors:0603,100kΩ
- added R9: 47kΩ, PCM_JLCPCB:R_0603, symbol PCM_JLCPCB-Resistors:0603,47kΩ
- added U2: AMS1117, PCM_JLCPCB:SOT-223-3_L6.5-W3.4-P2.30-LS7.0-BR, symbol PCM_JLCPCB-Power:LDO, 3.3V, 1A
- added U5, U7: LTV-827S, Package_DIP:SMDIP-8_W9.53mm, symbol Isolator:LTV-827S
Connections:
- net +3V3: now also C3.2, C6.1, U2.2 (VOUT), U2.4 (VOUT)
- net BEMF_U: now also R1.1
- net BEMF_V: now also R2.1
- net BEMF_W: now also R3.1
- net BEMF_X: now also R4.1
- net ETH_RXN: now also U1.64 (PC7)
- net ETH_RXP: now also U1.63 (PC6)
- net ETH_TXN: now also U1.66 (PC9)
- net ETH_TXP: now also U1.65 (PC8)
- net GND: now also C17.2, C3.1, C4.1, C5.2, C6.2, D8.2, D9.2, R10.2, R11.2, U2.1 (GND), U5.5, U5.7, U7.5, U7.7
- net LIM_H: now also U1.45 (PE14)
- net LIM_L: now also U1.44 (PE13)
- net PWMH0: now also U1.67 (PA8)
- net PWMH1: now also U1.68 (PA9)
- net PWMH2: now also U1.69 (PA10)
- net PWMH3: now also U1.93 (PB7)
- net PWML0: now also U1.39 (PE8)
- net PWML1: now also U1.41 (PE10)
- net PWML2: now also U1.43 (PE12)
- net PWML3: now also U1.35 (PB0)
- net SPI_MISO: now also U1.90 (PB4)
- net SPI_MOSI: now also U1.91 (PB5)
- net SPI_NSS: now also U1.77 (PA15)
- net SPI_SCK: now also U1.89 (PB3)
- net SYNC: now also U7.6
- net USBFS_N: now also U1.70 (PA11)
- net USBFS_P: now also U1.71 (PA12)
- net VBUS: now also R9.2
- net VBUS_MON: now reaches C37.2
- net VBUS_MON: now also U1.16 (PC1), D8.1, R10.1, R9.1
- net VGG_MON: now reaches U1.15 (PC0)
- net VGG_MON: now also C4.2, D9.1, R11.1, R12.2
- net OPA_O_X: now reaches U1.23 (PA0)
- net OPA_O_X: now also R8.1
- net OPA_O_W: now reaches U1.24 (PA1)
- net OPA_O_W: now also R7.1
- net OPA_O_V: now reaches U1.25 (PA2)
- net OPA_O_V: now also R6.1
- net OPA_O_U: now reaches U1.26 (PA3)
- net OPA_O_U: now also R5.1
- net ENC0_A: now reaches U1.3 (PE4)
- net U_I: now reaches U1.31 (PA6)
- net U_I: now also U1.32 (PA7)
- net BEMF_C: now reaches U1.36 (PB1)
- net BEMF_C: now also U1.37 (PB2), U1.47 (PB10), U1.48 (PB11)
- net ENC0_B: now reaches U1.4 (PE5)
- net STO_H: now reaches U1.46 (PE15)
- net STO_H: now also U5.6
- net ENC0_C: now reaches U1.5 (PE6)
- net at U1.51 (PB12): now also R4.2, R8.2
- net at U1.52 (PB13): now also R3.2, R7.2
- net at U1.53 (PB14): now also R2.2, R6.2
- net at U1.54 (PB15): now also R1.2, R5.2
- net CAN_RX: now reaches U1.81 (PD0)
- net CAN_TX: now reaches U1.82 (PD1)
- net STO_L: now reaches U1.96 (PB9)
- net STO_L: now also U5.8
- new net: J7.1, U5.1, U5.3
- new net: J7.2, R23.2
- new net: J7.3, R24.2
- new net: J7.4, U7.1, U7.3
- new net: J7.5, R31.2
- new net: J7.6, R32.2
- new net: C17.1, J7.S1 (SHIELD), J7.S2 (SHIELD__1)
- new net: R23.1, U5.4
- new net: R31.1, U7.4
- new net: R24.1, U5.2
- new net: R32.1, U7.2
- new net +5V: C5.1, R12.1, U2.3 (VIN)
- no-connect marks 0 -> 1
Other:
- removed sheet Gates+Fets
- added sheet 5vBuck (buck.kicad_sch)
- added sheet GANFETS (ganfets.kicad_sch)
- added sheet can (can.kicad_sch)
- added sheet encoder1 (encoder1.kicad_sch)
- sheet usb_c ports: added none; removed #PG_OD
- note added: "7,8,10 exti"
- note added: ">>UART5-TX >>UART5-RX"
- note removed: "1.5V Trigger OVP"
- note removed: "default rst>"
- moved on the sheet: C32, C33, C37, D1, D3, D4, J4, J5, R55, R60, R62, R63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
